Commit message: Initial commit

File: install/hospital_hardware/share/hospital_hardware/urdf/robot.urdf (robot description, URDF)
Before this commit: robot hospital_robot, 7 links, 6 joints
Links:
- removed link odom
Joints:
- removed joint odom_joint

File: src/hospital_hardware/urdf/robot.urdf (robot description, URDF)
Before this commit: robot hospital_robot, 7 links, 6 joints
Links:
- removed link odom
Joints:
- removed joint odom_joint
