Commit message: pi5 updated

File: src/hospital_hardware/urdf/robot.urdf (robot description, URDF)
Before this commit: robot hospital_robot, 6 links, 5 joints
Links:
- removed link lidar_link
- added link laser; visual cylinder length=0.05 radius=0.1
Joints:
- joint lidar_joint: child lidar_link -> laser
